File: power-sensor-breakout/power-sensor-breakout.kicad_sch (KiCad schematic)
At the start: 13 parts, among them J1 batt_1S, J10 INA219_breakout, J11 PH2.0-4P, J12 HY2.0, J13 100mil, J2 batt_1S, J3 batt_2S_PH, J4 batt_2S_254, J5 batt_2S, J6 batt_2S_PH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

Commit message: Add basic info
Other:
- title: (none) -> Battery to INA219 module to load
Changed lines of the file:
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@@
 (kicad_sch (version 20230121) (generator eeschema)
-  (paper "A4")
+  (paper "USLetter")
+  (title_block
+    (title "Battery to INA219 module to load")
+    (date "2023-06-18")
+    (comment 1 "Dan White")
+    (comment 2 "Electrical and Computer Engineering")
+    (comment 3 "Valparaiso University")
+  )
   (junction (at 119.38 67.31) (diameter 0) (color 0 0 0 0)
   )
